Commit message: little minor changes

File: urdf/mark2_helice_fixa.urdf (robot description, URDF)
Before this commit: robot mark2, 5 links, 4 joints
Links:
- link base_link: geometry collision mesh filename=package://sjtu-drone/meshes/helice_fixa/base_link.STL; visual mesh filename=package://sjtu-drone/meshes/Mark_2.dae

File: urdf/sjtu_drone.urdf (robot description, URDF)
Before this commit: robot sjtu_drone, 1 links, 0 joints
Links:
- link base_link: geometry collision mesh filename=package://sjtu-drone/meshes/quadrotor_4.stl; visual mesh filename=package://sjtu-drone/meshes/quadrotor_4.dae
